Commit message: update urdf file

File: urdf/ros_robot.urdf.xacro (robot description, xacro)
@@ -65,7 +65,28 @@
 		</collision>
 	</link>
-	<joint name="base_to_top_left_wheel" type="fixed">
-		<origin xyz="0.185 0.115 0.052"/>
+	<joint name="front_steer_joint" type="revolute">
+		<limit effort="100" lower="-1" upper="1" velocity="10"/>
+		<axis xyz="0 0 -1"/>
+		<origin xyz="0.185 0 0.052"/>
 		<parent link="base_link"/>
+		<child link="front_steer"/>
+	</joint>
+	<link name="front_steer">
+	</link>
+	<joint name="front_left_wheel_revolute_joint" type="revolute">
+		<limit effort="100" lower="-1" upper="1" velocity="10"/>
+		<axis xyz="0 0 1"/>
+		<origin rpy="0 0 0" xyz="0.185 0.115 0.052"/>
+		<mimic joint="front_steer_joint" multiplier="1.0"/>
+		<parent link="base_link"/>
+		<child link="front_left_wheel_revolute"/>
+	</joint>
+	<link name="front_left_wheel_revolute">
+	</link>
+	<joint name="base_to_top_left_wheel" type="continuous">
+		<origin rpy="0 0 0"/>
+		<axis xyz="0 1 0"/>
+		<mimic joint="base_to_bottom_left_wheel" multiplier="1.0"/>
+		<parent link="front_left_wheel_revolute"/>
 		<child link="top_left_wheel"/>
 	</joint>
@@ -85,7 +106,19 @@
 		</collision>
 	</link>
-	<joint name="base_to_top_right_wheel" type="fixed">
-		<origin xyz="0.185 -0.115 0.052"/>
+	<joint name="front_right_wheel_revolute_joint" type="revolute">
+		<limit effort="100" lower="-1" upper="1" velocity="10"/>
+		<axis xyz="0 0 1"/>
+		<origin rpy="0 0 0" xyz="0.185 -0.115 0.052"/>
+		<mimic joint="front_steer_joint" multiplier="1.0"/>
 		<parent link="base_link"/>
+		<child link="front_right_wheel_revolute"/>
+	</joint>
+	<link name="front_right_wheel_revolute">
+	</link>
+	<joint name="base_to_top_right_wheel" type="continuous">
+		<origin rpy="0 0 0"/>
+		<axis xyz="0 1 0"/>
+		<mimic joint="base_to_bottom_right_wheel" multiplier="1.0"/>
+		<parent link="front_right_wheel_revolute"/>
 		<child link="top_right_wheel"/>
 	</joint>
@@ -105,6 +138,16 @@
 		</collision>
 	</link>
-	<joint name="base_to_bottom_left_wheel" type="fixed">
-		<origin xyz="-0.145 0.115 0.052"/>
+	<joint name="rear_wheel_joint" type="continuous">
+		<axis xyz="0 1 0"/>
+		<origin rpy="0 0 0" xyz="-0.145 0 0.052"/>
+		<parent link="base_link"/>
+		<child link="rear_steer"/>
+	</joint>
+	<link name="rear_steer">
+	</link>
+	<joint name="base_to_bottom_left_wheel" type="continuous">
+		<axis xyz="0 0 1"/>
+		<origin rpy="-1.5708 0 0" xyz="-0.145 0.115 0.052"/>
+		<mimic joint="rear_wheel_joint" multiplier="1.0"/>
 		<parent link="base_link"/>
 		<child link="bottom_left_wheel"/>
@@ -112,5 +155,4 @@
 	<link name="bottom_left_wheel">
 		<visual>
-			<origin rpy="1.5708 0 0"/>
 			<geometry>
 				<cylinder length="0.045" radius="0.052"/>
@@ -119,5 +161,4 @@
 		</visual>
 		<collision>
-			<origin rpy="1.5708 0 0"/>
 			<geometry>
 				<cylinder length="0.045" radius="0.052"/>
@@ -125,6 +166,8 @@
 		</collision>
 	</link>
-	<joint name="base_to_bottom_right_wheel" type="fixed">
-		<origin xyz="-0.145 -0.115 0.052"/>
+	<joint name="base_to_bottom_right_wheel" type="continuous">
+		<axis xyz="0 0 1"/>
+		<origin rpy="-1.5708 0 0" xyz="-0.145 -0.115 0.052"/>
+		<mimic joint="rear_wheel_joint" multiplier="1.0"/>
 		<parent link="base_link"/>
 		<child link="bottom_right_wheel"/>
@@ -132,5 +175,4 @@
 	<link name="bottom_right_wheel">
 		<visual>
-			<origin rpy="1.5708 0 0"/>
 			<geometry>
 				<cylinder length="0.045" radius="0.052"/>
@@ -139,5 +181,4 @@
 		</visual>
 		<collision>
-			<origin rpy="1.5708 0 0"/>
 			<geometry>
 				<cylinder length="0.045" radius="0.052"/>

Commit message: add wheel model in urdf file

File: urdf/ros_robot.urdf.xacro (robot description, xacro)
@@ -10,4 +10,9 @@
 		<color rgba="0.3 0.3 0.3 1.0"/>
 	</material>
+	<xacro:macro name="wheel">
+		<geometry>
+			<mesh filename="package://mobile/car_parts/rviz/wheel.stl" scale="0.001 0.001 0.001"/>
+		</geometry>
+	</xacro:macro>
 	<link name="base_link">
 		<visual>
@@ -26,5 +31,5 @@
 	</link>
 	<joint name="base_to_laser" type="fixed">
-		<origin xyz="0.06 0.13 -0.545"/>
+		<origin xyz="-0.045 0 0"/>
 		<parent link="base_link"/>
 		<child link="laser"/>
@@ -32,5 +37,5 @@
 	<link name="laser">
 		<visual>
-			<origin rpy="1.5708 0 0"/>
+			<origin rpy="1.5708 0 0" xyz="0.06 0.13 -0.545"/>
 			<geometry>
 				<mesh filename="package://mobile/car_parts/rviz/rplidar-a1.stl" scale="0.001 0.001 0.001"/>
@@ -93,15 +98,11 @@
 	<link name="top_left_wheel">
 		<visual>
-			<origin rpy="1.5708 0 0"/>
-			<geometry>
-				<cylinder length="0.045" radius="0.052"/>
-			</geometry>
+			<origin rpy="-1.5708 0 0"/>
+			<wheel/>
 			<material name="gray"/>
 		</visual>
 		<collision>
-			<origin rpy="1.5708 0 0"/>
-			<geometry>
-				<cylinder length="0.045" radius="0.052"/>
-			</geometry>
+			<origin rpy="-1.5708 0 0"/>
+			<wheel/>
 		</collision>
 	</link>
@@ -125,15 +126,11 @@
 	<link name="top_right_wheel">
 		<visual>
-			<origin rpy="1.5708 0 0"/>
-			<geometry>
-				<cylinder length="0.045" radius="0.052"/>
-			</geometry>
+			<origin rpy="1.5708 3.14 0"/>
+			<wheel/>
 			<material name="gray"/>
 		</visual>
 		<collision>
-			<origin rpy="1.5708 0 0"/>
-			<geometry>
-				<cylinder length="0.045" radius="0.052"/>
-			</geometry>
+			<origin rpy="1.5708 3.14 0"/>
+			<wheel/>
 		</collision>
 	</link>
@@ -155,18 +152,14 @@
 	<link name="bottom_left_wheel">
 		<visual>
-			<geometry>
-				<cylinder length="0.045" radius="0.052"/>
-			</geometry>
+			<wheel/>
 			<material name="gray"/>
 		</visual>
 		<collision>
-			<geometry>
-				<cylinder length="0.045" radius="0.052"/>
-			</geometry>
+			<wheel/>
 		</collision>
 	</link>
 	<joint name="base_to_bottom_right_wheel" type="continuous">
-		<axis xyz="0 0 1"/>
-		<origin rpy="-1.5708 0 0" xyz="-0.145 -0.115 0.052"/>
+		<axis xyz="0 0 -1"/>
+		<origin rpy="1.5708 3.14 0" xyz="-0.145 -0.115 0.052"/>
 		<mimic joint="rear_wheel_joint" multiplier="1.0"/>
 		<parent link="base_link"/>
@@ -175,13 +168,9 @@
 	<link name="bottom_right_wheel">
 		<visual>
-			<geometry>
-				<cylinder length="0.045" radius="0.052"/>
-			</geometry>
+			<wheel/>
 			<material name="gray"/>
 		</visual>
 		<collision>
-			<geometry>
-				<cylinder length="0.045" radius="0.052"/>
-			</geometry>
+			<wheel/>
 		</collision>
 	</link>

Commit message: update urdf file

File: urdf/ros_robot.urdf.xacro (robot description, xacro)
@@ -17,5 +17,5 @@
 	<link name="base_link">
 		<visual>
-			<origin rpy="0 0 -1.5708" xyz="0 0.1375 0.048"/>
+			<origin rpy="0 0 -1.5708" xyz="0.145 0.1375 0.048"/>
 			<geometry>
 				<mesh filename="package://mobile/car_parts/rviz/car-body.stl" scale="0.001 0.001 0.001"/>
@@ -24,5 +24,5 @@
 		</visual>
 		<collision>
-			<origin rpy="0 0 -1.5708" xyz="0 0.1375 0.048"/>
+			<origin rpy="0 0 -1.5708" xyz="0.145 0.1375 0.048"/>
 			<geometry>
 				<mesh filename="package://mobile/car_parts/rviz/car-body.stl" scale="0.001 0.001 0.001"/>
@@ -31,5 +31,5 @@
 	</link>
 	<joint name="base_to_laser" type="fixed">
-		<origin xyz="-0.045 0 0"/>
+		<origin xyz="0.1 0 0"/>
 		<parent link="base_link"/>
 		<child link="laser"/>
@@ -37,5 +37,5 @@
 	<link name="laser">
 		<visual>
-			<origin rpy="1.5708 0 0" xyz="0.06 0.13 -0.545"/>
+			<origin rpy="1.5708 0 0" xyz="0.10 0.13 -0.545"/>
 			<geometry>
 				<mesh filename="package://mobile/car_parts/rviz/rplidar-a1.stl" scale="0.001 0.001 0.001"/>
@@ -44,5 +44,5 @@
 		</visual>
 		<collision>
-			<origin rpy="1.5708 0 0"/>
+			<origin rpy="1.5708 0 0" xyz="0.10 0.13 -0.545"/>
 			<geometry>
 				<mesh filename="package://mobile/car_parts/rviz/rplidar-a1.stl" scale="0.001 0.001 0.001"/>
@@ -51,5 +51,5 @@
 	</link>
 	<joint name="base_to_camera" type="fixed">
-		<origin xyz="0.265 0 0.12"/>
+		<origin xyz="0.41 0 0.12"/>
 		<parent link="base_link"/>
 		<child link="camera"/>
@@ -73,5 +73,5 @@
 		<limit effort="100" lower="-1" upper="1" velocity="10"/>
 		<axis xyz="0 0 -1"/>
-		<origin xyz="0.185 0 0.052"/>
+		<origin xyz="0.33 0 0.052"/>
 		<parent link="base_link"/>
 		<child link="front_steer"/>
@@ -82,5 +82,5 @@
 		<limit effort="100" lower="-1" upper="1" velocity="10"/>
 		<axis xyz="0 0 1"/>
-		<origin rpy="0 0 0" xyz="0.185 0.115 0.052"/>
+		<origin rpy="0 0 0" xyz="0.33 0.115 0.052"/>
 		<mimic joint="front_steer_joint" multiplier="1.0"/>
 		<parent link="base_link"/>
@@ -110,5 +110,5 @@
 		<limit effort="100" lower="-1" upper="1" velocity="10"/>
 		<axis xyz="0 0 1"/>
-		<origin rpy="0 0 0" xyz="0.185 -0.115 0.052"/>
+		<origin rpy="0 0 0" xyz="0.33 -0.115 0.052"/>
 		<mimic joint="front_steer_joint" multiplier="1.0"/>
 		<parent link="base_link"/>
@@ -137,5 +137,5 @@
 	<joint name="rear_wheel_joint" type="continuous">
 		<axis xyz="0 1 0"/>
-		<origin rpy="0 0 0" xyz="-0.145 0 0.052"/>
+		<origin rpy="0 0 0" xyz="0 0 0.052"/>
 		<parent link="base_link"/>
 		<child link="rear_steer"/>
@@ -145,5 +145,5 @@
 	<joint name="base_to_bottom_left_wheel" type="continuous">
 		<axis xyz="0 0 1"/>
-		<origin rpy="-1.5708 0 0" xyz="-0.145 0.115 0.052"/>
+		<origin rpy="-1.5708 0 0" xyz="0 0.115 0.052"/>
 		<mimic joint="rear_wheel_joint" multiplier="1.0"/>
 		<parent link="base_link"/>
@@ -161,5 +161,5 @@
 	<joint name="base_to_bottom_right_wheel" type="continuous">
 		<axis xyz="0 0 -1"/>
-		<origin rpy="1.5708 3.14 0" xyz="-0.145 -0.115 0.052"/>
+		<origin rpy="1.5708 3.14 0" xyz="0 -0.115 0.052"/>
 		<mimic joint="rear_wheel_joint" multiplier="1.0"/>
 		<parent link="base_link"/>

Commit message: update urdf file

File: urdf/ros_robot.urdf.xacro (robot description, xacro)
@@ -31,22 +31,9 @@
 	</link>
 	<joint name="base_to_laser" type="fixed">
-		<origin xyz="0.1 0 0"/>
+		<origin xyz="0.123 0 0"/>
 		<parent link="base_link"/>
 		<child link="laser"/>
 	</joint>
 	<link name="laser">
-		<visual>
-			<origin rpy="1.5708 0 0" xyz="0.10 0.13 -0.545"/>
-			<geometry>
-				<mesh filename="package://mobile/car_parts/rviz/rplidar-a1.stl" scale="0.001 0.001 0.001"/>
-			</geometry>
-			<material name="black"/>
-		</visual>
-		<collision>
-			<origin rpy="1.5708 0 0" xyz="0.10 0.13 -0.545"/>
-			<geometry>
-				<mesh filename="package://mobile/car_parts/rviz/rplidar-a1.stl" scale="0.001 0.001 0.001"/>
-			</geometry>
-		</collision>
 	</link>
 	<joint name="base_to_camera" type="fixed">
@@ -70,8 +57,15 @@
 		</collision>
 	</link>
+	<joint name="base_to_imu" type="fixed">
+		<origin rpy="0 0 0" xyz="0.307 0 0.12"/>
+		<parent link="base_link"/>
+		<child link="imu_link"/>
+	</joint>
+	<link name="imu_link">
+	</link>
 	<joint name="front_steer_joint" type="revolute">
 		<limit effort="100" lower="-1" upper="1" velocity="10"/>
 		<axis xyz="0 0 -1"/>
-		<origin xyz="0.33 0 0.052"/>
+		<origin xyz="0.326 0 0.052"/>
 		<parent link="base_link"/>
 		<child link="front_steer"/>
@@ -82,5 +76,5 @@
 		<limit effort="100" lower="-1" upper="1" velocity="10"/>
 		<axis xyz="0 0 1"/>
-		<origin rpy="0 0 0" xyz="0.33 0.115 0.052"/>
+		<origin rpy="0 0 0" xyz="0.326 0.115 0.052"/>
 		<mimic joint="front_steer_joint" multiplier="1.0"/>
 		<parent link="base_link"/>
@@ -99,10 +93,10 @@
 		<visual>
 			<origin rpy="-1.5708 0 0"/>
-			<wheel/>
+			<xacro:wheel/>
 			<material name="gray"/>
 		</visual>
 		<collision>
 			<origin rpy="-1.5708 0 0"/>
-			<wheel/>
+			<xacro:wheel/>
 		</collision>
 	</link>
@@ -110,5 +104,5 @@
 		<limit effort="100" lower="-1" upper="1" velocity="10"/>
 		<axis xyz="0 0 1"/>
-		<origin rpy="0 0 0" xyz="0.33 -0.115 0.052"/>
+		<origin rpy="0 0 0" xyz="0.326 -0.115 0.052"/>
 		<mimic joint="front_steer_joint" multiplier="1.0"/>
 		<parent link="base_link"/>
@@ -127,10 +121,10 @@
 		<visual>
 			<origin rpy="1.5708 3.14 0"/>
-			<wheel/>
+			<xacro:wheel/>
 			<material name="gray"/>
 		</visual>
 		<collision>
 			<origin rpy="1.5708 3.14 0"/>
-			<wheel/>
+			<xacro:wheel/>
 		</collision>
 	</link>
@@ -152,9 +146,9 @@
 	<link name="bottom_left_wheel">
 		<visual>
-			<wheel/>
+			<xacro:wheel/>
 			<material name="gray"/>
 		</visual>
 		<collision>
-			<wheel/>
+			<xacro:wheel/>
 		</collision>
 	</link>
@@ -168,9 +162,9 @@
 	<link name="bottom_right_wheel">
 		<visual>
-			<wheel/>
+			<xacro:wheel/>
 			<material name="gray"/>
 		</visual>
 		<collision>
-			<wheel/>
+			<xacro:wheel/>
 		</collision>
 	</link>
